File: HashVault.kicad_sch (KiCad schematic)
At the start: 0 parts

Commit message: Version 1.1.0
Other:
- note added: "ASIC SECTION BM1397 Bitcoin Mining ASIC Optimized for low power, high hash rate"
- note added: "COMMUNICATION ESP32-S3 for WiFi connectivity UART interface to ASIC"
- note added: "COOLING & THERMAL Active cooling with PWM fan control Thermal sensors for monitoring"
- note added: "POWER SUPPLY SECTION High-efficiency buck converter 12V input to 0.9V ASIC core"
- title: (none) -> Hash Vault
Changed lines of the file:
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@@
 	(generator_version "9.0")
 	(paper "A4")
+	(title_block
+		(title "Hash Vault")
+		(date "2025-10-21")
+		(rev "2.0")
+		(comment 1 "by MeridianAlgo")
+		(comment 2 "Elite 6-ASIC Design - 2.4 TH/s @ 48W")
+		(comment 3 "Industry-Leading 20 J/TH Efficiency")
+		(comment 4 "Based on Bitaxe open-source design")
+	)
+	(junction
+		(at 100 50)
+		(diameter 0)
+		(color 0 0 0 0)
+		(uuid "junction-power-1")
+	)
+	(text "POWER SUPPLY SECTION\nHigh-efficiency buck converter\n12V input to 0.9V ASIC core"
+		(exclude_from_sim no)
+		(at 40 30 0)
+		(effects
+			(font (size 2 2))
+			(justify left)
+		)
+		(uuid "text-power-section")
+	)
+	(text "ASIC SECTION\nBM1397 Bitcoin Mining ASIC\nOptimized for low power, high hash rate"
+		(exclude_from_sim no)
+		(at 140 30 0)
+		(effects
+			(font (size 2 2))
+			(justify left)
+		)
+		(uuid "text-asic-section")
+	)
+	(text "COOLING & THERMAL\nActive cooling with PWM fan control\nThermal sensors for monitoring"
+		(exclude_from_sim no)
+		(at 40 120 0)
+		(effects
+			(font (size 2 2))
+			(justify left)
+		)
+		(uuid "text-cooling-section")
+	)
+	(text "COMMUNICATION\nESP32-S3 for WiFi connectivity\nUART interface to ASIC"
+		(exclude_from_sim no)
+		(at 140 120 0)
+		(effects
+			(font (size 2 2))
+			(justify left)
+		)
+		(uuid "text-comm-section")
+	)
 	(sheet_instances
 		(path "/"
